File: zmigavac.kicad_pcb (KiCad board)
At the start: 2 copper layers, 154 x 123 mm, 61 parts, among them Q1 BC547, SW1 SW_SPDT, SW2 SW_DPST_x2, U1 NE555P, U2 74HC595, U3 ULN2803A, U5 TSR_1-2450

Commit message: Nova izmena
Parts:
- BT1: renamed from + BT1 -; value + Battery_Cell - -> Battery_Cell
Changed lines of the file:
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@@
 		(descr "terminal block MaiXu MX126-5.0-02P, 2 pins, pitch 5mm, size 10.5x7.8mm, drill diameter 1.3mm, pad diameter 2.8mm, https://www.lcsc.com/datasheet/lcsc_datasheet_2309150913_MAX-MX126-5-0-03P-GN01-Cu-S-A_C5188435.pdf")
 		(tags "THT terminal block MaiXu MX126-5.0-02P pitch 5mm size 10.5x7.8mm drill 1.3mm pad 2.8mm")
-		(property "Reference" "+ BT1 -"
+		(property "Reference" "BT1"
 			(at 2.25 -5.12 0)
 			(layer "F.SilkS")
@@
 			)
 		)
-		(property "Value" "+ Battery_Cell -"
+		(property "Value" "Battery_Cell"
 			(at 2.25 4.92 0)
 			(layer "F.Fab")
